File: circuitos/circuito control/circuito.kicad_pcb (KiCad board)
At the start: 2 copper layers, 27 parts, among them CON1 SD_Card, IC1 ATMEGA328-P, P1 CONN_5V, P2 CONN_02X03, P3 CONN_UART_USB, P4 CONN_UART, SW1 B_RST_N_O, SW2 B_SEL_N_O, SW3 B_CHG_N_O, Y1 16Mhz

Commit message: adapto graficos para el informe
Parts:
- C2: value 10n -> 100n
- moved P1 76.3 mm to (90.0, 102.5), turned to 180 degrees
- moved P3 74.0 mm to (117.5, 127.5), turned to 270 degrees
- moved C1 73.6 mm to (100.0, 120.0), turned to 180 degrees
- moved R1 72.9 mm to (95.0, 110.0), turned to 0 degrees
- moved R4 71.6 mm to (95.0, 72.5), turned to 270 degrees
- moved SW1 69.7 mm to (100.0, 115.0), turned to 270 degrees
- moved P4 67.5 mm to (100.0, 127.5), turned to 90 degrees
- moved IC1 63.7 mm to (100.0, 105.0), turned to 90 degrees
- moved Y1 53.0 mm to (120.0, 120.0), turned to 180 degrees
- moved SW2 52.6 mm to (130.0, 125.0), turned to 0 degrees
- moved SW3 50.6 mm to (135.0, 125.0), turned to 0 degrees
- moved C4 47.6 mm to (117.5, 112.5), turned to 180 degrees
- moved C3 40.3 mm to (125.0, 112.5), turned to 180 degrees
- moved P2 38.1 mm to (117.5, 80.0), turned to 90 degrees
- moved DS1 36.1 mm to (137.5, 65.0), turned to 270 degrees
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Connections:
- IC1 pad 2: /Rx_pc -> /Rx_int
- IC1 pad 3: /RX_USB -> /Tx_int
- IC1 pad 5: /Rx_int -> /Rx_pc
- IC1 pad 6: /Tx_int -> /RX_USB
Routing:
- net GND: track 415.4 -> 410.4 mm
- net /Rx_int: track 28.9 -> 25.2 mm
- net /Tx_int: track 27.6 -> 25.0 mm
- net /Rx_pc: track 25.0 -> 26.0 mm
